File: hardware/badge-44con-2025/badge-44con-2025.kicad_sch (KiCad schematic)
At the start: 8 parts, among them J1 Conn_01x04, SW1 SW_Nidec_CAS-120A1

Commit message: feat(Hw): Finished_SCH
Parts:
- added BT5, BT6, BT7: Battery_Cell, Battery:BatteryHolder_Keystone_2466_1xAAA, symbol Device:Battery_Cell
- added D7: LED, LED_SMD:LED_0603_1608Metric, symbol Device:LED
- added R4: 1k, Resistor_SMD:R_0603_1608Metric, symbol Device:R_Small
- BZ1: manf# (none) -> https://www.amazon.com/Cylewet-Terminals-Electronic-Electro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; provedor (none) -> Amazon
- J1: value Conn_01x04 -> 128x64 OLED Display; manf# (none) -> https://www.amazon.com/gp/product/B0D2RLXLBZ; provedor (none) -> Amazon
- JP1: #LCSC (none) -> ---; provedor (none) -> ---
- RV1: manf# (none) -> https://www.amazon.com/gp/product/B0CSW6D1N4; provedor (none) -> Amazon
- SW1: manf# (none) -> https://www.amazon.com/gp/product/B007QAJUUS; provedor (none) -> Amazon
- U1: value ~ -> AD8317_Module; manf# (none) -> https://www.amazon.com/gp/product/B07FHZXTCZ; provedor (none) -> Amazon
- U2: value ~ -> MT3608_Boost_converter; manf# (none) -> https://www.amazon.com/gp/product/B09S8ZDVBN; provedor (none) -> Amazon
- U3: value ~ -> ESP32-WEMOS D1 mini; manf# (none) -> https://a.co/d/5juHR3B; provedor (none) -> Amazon
Connections:
- net +3.3V: now also RV1.1
- net +5V: now also R4.2; no longer RV1.1
- net +5VP: now also BT7.1 (+)
- net GND: now also BT6.2 (-), D7.1 (K)
- new net: BT5.1 (+), BT7.2 (-)
- new net: D7.2 (A), R4.1
- new net: BT5.2 (-), BT6.1 (+)
Other:
- note added: "BATTERY"
- note removed: "AD8317_Module"
- note removed: "MT3608_Module"
- moved on the sheet: BZ1, J1, U2, U3
