File: hardware/badge-44con-2025/badge-44con-2025.kicad_sch (KiCad schematic)
At the start: 13 parts, among them J1 128x64 OLED Display, SW1 SW_Nidec_CAS-120A1, U1 AD8317_Module, U2 MT3608_Boost_converter, U3 ESP32-WEMOS D1 mini

Commit message: feat(Hw): floorplan_draft
Parts:
- JP1: footprint (none) -> Connector_PinHeader_2.54mm:PinHeader_1x02_P2.54mm_Vertical
- RV1: footprint (none) -> Potentiometer_THT:Potentiometer_Alps_RK163_Single_Horizontal
- U2: footprint (none) -> badge-44con-2025:MT3608
- U3: footprint (none) -> badge-44con-2025:Wemos Mini D1 ESP WiFi + Bluetooth CP2104
Changed lines of the file:
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@@
 			)
 		)
-		(property "Footprint" ""
+		(property "Footprint" "badge-44con-2025:Wemos Mini D1 ESP WiFi + Bluetooth CP2104"
 			(at 54.61 48.26 0)
 			(effects
@@
 			)
 		)
-		(property "Footprint" ""
+		(property "Footprint" "Connector_PinHeader_2.54mm:PinHeader_1x02_P2.54mm_Vertical"
 			(at 237.49 67.31 0)
 			(effects
@@
 			)
 		)
-		(property "Footprint" ""
+		(property "Footprint" "badge-44con-2025:MT3608"
 			(at 148.59 35.56 0)
 			(effects
@@
 			)
 		)
-		(property "Footprint" ""
+		(property "Footprint" "Potentiometer_THT:Potentiometer_Alps_RK163_Single_Horizontal"
 			(at 93.98 27.94 0)
 			(effects

Commit message: feat(Hw):Added_microcontroller
Parts:
- added C1 (x2): .1uF, Capacitor_SMD:C_0603_1608Metric, symbol Device:C_Small
- added D1, D2, D3, D4, D5: LED, LED_SMD:LED_0603_1608Metric, symbol Device:LED
- added D1, D6: R_LED, Unknown:LYT77K-K2M1, symbol Device:LED
- added J2: Conn_02x03_Odd_Even, Connector_PinHeader_2.54mm:PinHeader_2x03_P2.54mm_Vertical_SMD, symbol Connector_Generic:Conn_02x03_Odd_Even
- added R1 (x2), R2, R3, R5, R6, R7: 220, Resistor_SMD:R_0603_1608Metric, symbol Device:R_Small
- added SW2: RESET, Button_Switch_SMD:SW_SPST_TL3342, symbol Switch:SW_Push
- added U5: CH32V003FxPx, Package_SO:TSSOP-20_4.4x6.5mm_P0.65mm, symbol MCU_WCH_CH32V0:CH32V003FxPx
Connections:
- net +3.3V: now also C1.2, J2.5 (Pin_5), U5.9 (VDD)
- net GND: now also C1.1, C1.1, J2.6 (Pin_6), R1.2, R1.2, R2.2, R3.2, R5.2, R6.2, R7.2, SW2.1, U5.7 (VSS)
- net SCL: now also U5.12 (PC2)
- net SDA: now also U5.11 (PC1)
- new net: D5.1 (K), R5.1
- new net: D4.1 (K), R1.1
- new net: D6.1 (K), R6.1
- new net: D2.1 (K), R2.1
- new net: D3.1 (K), R3.1
- new net: D1.1 (K), R7.1
- new net: D1.1 (K), R1.1
- new net DOWN: U5.6 (PA2)
- new net LED1: D1.2 (A), U5.20 (PD3)
- new net LED2: D2.2 (A), U5.2 (PD5)
- new net LED3: D3.2 (A), U5.1 (PD4)
- new net LED4: D4.2 (A), U5.5 (PA1)
- new net LED5: D5.2 (A), U5.19 (PD2)
- new net LED6: D6.2 (A), U5.15 (PC5)
- new net LED7: D1.2 (A), U5.10 (PC0)
- new net LEFT: U5.13 (PC3)
- new net RIGHT: U5.8 (PD0)
- new net RST: C1.2, SW2.2, U5.4 (PD7)
- new net SWDIO: J2.2 (Pin_2), U5.18 (PD1)
- new net UP: U5.14 (PC4)
- no-connect marks 28 -> 34

Commit message: fix(Hw): Changed_PCB_design
Parts:
- removed D1, D6: R_LED, Unknown:LYT77K-K2M1, symbol Device:LED
- removed D5: LED, LED_SMD:LED_0603_1608Metric, symbol Device:LED
- removed R5, R6, R7: 220, Resistor_SMD:R_0603_1608Metric, symbol Device:R_Small
- RV1: footprint Potentiometer_THT:Potentiometer_Alps_RK163_Single_Horizontal -> badge-44con-2025:Potentiometer_generic
- renumbered BT7 to BT1, BT5 to BT2, BT6 to BT3, C1 to C2, D7 to D1, D1 to D2, D2 to D3, D3 to D4, D4 to D5, R4 to R1, R1 to R2, R2 to R3, R3 to R4, R1 to R5, SW2 to SW1, SW1 to SW2, U3 to U1, U5 to U2, U2 to U3, U1 to U4
Connections:
- net GND: no longer R2.2, R3.2, R4.2, R5.2
- net SCL: no longer J1.2 (Pin_2), U1.23 (PIN_22)
- net SDA: no longer J1.1 (Pin_1), U1.24 (PIN_21)
- net DOWN: no longer names the net of U2.6 (PA2)
- net LEFT: no longer names the net of U2.13 (PC3)
- net RIGHT: no longer names the net of U2.8 (PD0)
- net UP: no longer names the net of U2.14 (PC4)
- new net: R2.2, R3.2, R4.2, R5.2
- new net SCL_ESP: J1.2 (Pin_2), U1.23 (PIN_22)
- new net SDA_ESP: J1.1 (Pin_1), U1.24 (PIN_21)
- no-connect marks 34 -> 38

Commit message: feat(Hw): Started routing
Connections:
- net LED5: no longer names the net of U2.19 (PD2)
- net LED6: no longer names the net of U2.15 (PC5)
- net LED7: no longer names the net of U2.10 (PC0)
- no-connect marks 38 -> 41
Changed lines of the file:
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@@
+	)
+	(no_connect
+		(at 59.69 154.94)
 	)
 	(no_connect
@@
 	)
 	(no_connect
+		(at 59.69 167.64)
+	)
+	(no_connect
 		(at 44.45 35.56)
 	)
 	(no_connect
 		(at 44.45 50.8)
+	)
+	(no_connect
+		(at 88.9 160.02)
 	)
 	(no_connect
@@
 		)
 	)
-	(label "LED5"
-		(at 88.9 160.02 0)
-		(effects
-			(font
-				(size 1.27 1.27)
-			)
-			(justify left bottom)
-		)
-	)
 	(label "LED"
 		(at 160.02 62.23 0)
@@
 		)
 	)
-	(label "LED7"
-		(at 59.69 154.94 180)
-		(effects
-			(font
-				(size 1.27 1.27)
-			)
-			(justify right bottom)
-		)
-	)
 	(label "LED1"
 		(at 88.9 162.56 0)
@@
 		)
 	)
-	(label "LED6"
-		(at 59.69 167.64 180)
-		(effects
-			(font
-				(size 1.27 1.27)
-			)
-			(justify right bottom)
-		)
-	)

Commit message: feat(Hw): finished_routing
Parts:
- added JP2, JP3: Jumper_3_Open, Jumper:SolderJumper-3_P1.3mm_Open_RoundedPad1.0x1.5mm, symbol Jumper:Jumper_3_Open
Connections:
- net GND: now also R2.2, R3.2, R4.2, R5.2
- net LED1: now also U2.2 (PD5); no longer U2.20 (PD3)
- net LED2: now also U2.1 (PD4); no longer U2.2 (PD5)
- net LED3: now also U2.3 (PD6); no longer U2.1 (PD4)
- net SCL: now also J1.2 (Pin_2), JP3.2 (C); no longer U2.12 (PC2)
- net SCL_ESP: now also JP3.3 (B); no longer J1.2 (Pin_2)
- net SDA: now also J1.1 (Pin_1), JP2.2 (C); no longer U2.11 (PC1)
- net SDA_ESP: now also JP2.3 (B); no longer J1.1 (Pin_1)
- new net CH3_SCL: JP3.1 (A), U2.12 (PC2)
- new net CH3_SDA: JP2.1 (A), U2.11 (PC1)
Other:
- moved on the sheet: J2

Commit message: fix(Hw):fixed_BOM
Parts:
- D2: #LCSC (none) -> C965812; LCSC# C434424 -> C965812
- D3: #LCSC (none) -> C205441; LCSC# C434424 -> C205441
- D4: #LCSC (none) -> C965815; LCSC# C434424 -> C965815
- D5: #LCSC (none) -> C84261; LCSC# C434424 -> C84261
- J2: #LCSC (none) -> C3975148
- R2, R3, R4, R5: #LCSC (none) -> C22962
- SW1: #LCSC (none) -> C318889
- U2: #LCSC (none) -> C5187096
Changed lines of the file:
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@@
 			)
 		)
-		(property "LCSC#" "C434424"
+		(property "LCSC#" "C84261"
 			(at 220.98 119.38 0)
 			(effects
@@
 			)
 		)
+		(property "#LCSC" "C84261"
+			(at 220.98 119.38 0)
+			(effects
+				(font
+					(size 1.27 1.27)
+				)
+			)
+		)
 		(pin "1"
 		)
@@
 			)
 		)
+		(property "#LCSC" "C22962"
+			(at 210.82 119.38 0)
+			(effects
+				(font
+					(size 1.27 1.27)
+				)
+			)
+		)
 		(pin "1"
 		)
@@
 			)
 		)
+		(property "#LCSC" "C5187096"
+			(at 74.93 167.64 0)
+			(effects
+				(font
+					(size 1.27 1.27)
+				)
+			)
+		)
 		(pin "4"
 		)
@@
 			)
 		)
-		(property "LCSC#" "C434424"
+		(property "LCSC#" "C205441"
 			(at 220.98 104.14 0)
 			(effects
@@
 			)
 		)
+		(property "#LCSC" "C205441"
+			(at 220.98 104.14 0)
+			(effects
+				(font
+					(size 1.27 1.27)
+				)
+			)
+		)
 		(pin "1"
 		)
@@
 			)
 		)
-		(property "LCSC#" "C434424"
+		(property "LCSC#" "C965815"
 			(at 220.98 111.76 0)
 			(effects
@@
 			)
 		)
+		(property "#LCSC" "C965815"
+			(at 220.98 111.76 0)
+			(effects
+				(font
+					(size 1.27 1.27)
+				)
+			)
+		)
 		(pin "1"
 		)
@@
 			)
 		)
+		(property "#LCSC" "C318889"
+			(at 109.093 178.308 0)
+			(effects
+				(font
+					(size 1.27 1.27)
+				)
+			)
+		)
 		(pin "1"
 		)
@@
 			)
 		)
+		(property "#LCSC" "C22962"
+			(at 210.82 111.76 0)
+			(effects
+				(font
+					(size 1.27 1.27)
+				)
+			)
+		)
 		(pin "1"
 		)
@@
 			)
 		)
-		(property "LCSC#" "C434424"
+		(property "LCSC#" "C965812"
 			(at 220.98 96.52 0)
 			(effects
@@
 			)
 		)
+		(property "#LCSC" "C965812"
+			(at 220.98 96.52 0)
+			(effects
+				(font
+					(size 1.27 1.27)
+				)
+			)
+		)
 		(pin "1"
 		)
@@
 			)
 		)
+		(property "#LCSC" "C22962"
+			(at 210.82 96.52 0)
+			(effects
+				(font
+					(size 1.27 1.27)
+				)
+			)
+		)
 		(pin "1"
 		)
@@
 			)
 		)
+		(property "#LCSC" "C22962"
+			(at 210.82 104.14 0)
+			(effects
+				(font
+					(size 1.27 1.27)
+				)
+			)
+		)
 		(pin "1"
 		)
@@
 			)
 		)
+		(property "#LCSC" "C3975148 "
+			(at 33.02 139.7 0)
+			(effects
+				(font
+					(size 1.27 1.27)
+				)
+			)
+		)

Commit message: feat(Hw):Added_labels_and_changed_switch
Parts:
- JP2, JP3: footprint Jumper:SolderJumper-3_P1.3mm_Open_RoundedPad1.0x1.5mm -> Jumper:SolderJumper-3_P1.3mm_Bridged2Bar12_RoundedPad1.0x1.5mm
- SW2: footprint badge-44con-2025:a12013100ux0116 -> badge-44con-2025:JS102011SAQN; #LCSC (none) -> C221660; manf# https://www.amazon.com/gp/product/B007QAJUUS -> (none)
Changed lines of the file:
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@@
 			)
 		)
-		(property "Footprint" "badge-44con-2025:a12013100ux0116"
+		(property "Footprint" "badge-44con-2025:JS102011SAQN"
 			(at 148.59 74.93 0)
 			(effects
@@
 			)
 		)
-		(property "manf#" "https://www.amazon.com/gp/product/B007QAJUUS"
+		(property "manf#" ""
 			(at 147.828 52.832 0)
+			(effects
+				(font
+					(size 1.27 1.27)
+				)
+				(hide yes)
+			)
+		)
+		(property "#LCSC" "C221660"
+			(at 139.446 66.548 0)
 			(effects
 				(font
@@
 			)
 		)
-		(property "Footprint" "Jumper:SolderJumper-3_P1.3mm_Open_RoundedPad1.0x1.5mm"
+		(property "Footprint" "Jumper:SolderJumper-3_P1.3mm_Bridged2Bar12_RoundedPad1.0x1.5mm"
 			(at 35.56 166.37 0)
 			(effects
@@
 			)
 		)
-		(property "Footprint" "Jumper:SolderJumper-3_P1.3mm_Open_RoundedPad1.0x1.5mm"
+		(property "Footprint" "Jumper:SolderJumper-3_P1.3mm_Bridged2Bar12_RoundedPad1.0x1.5mm"
 			(at 36.83 182.88 0)
 			(effects

Commit message: fix(Hw):Fixed_switch_in_BOM
Parts:
- SW2: provedor Amazon -> LCSC
Changed lines of the file:
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@@
 			)
 		)
-		(property "provedor" "Amazon"
+		(property "provedor" "LCSC"
 			(at 142.494 65.786 0)
 			(effects
