File: hardware/badge-44con-2025/badge-44con-2025.kicad_pcb (KiCad board)
At the start: 2 copper layers, 80.2 x 100 mm, 13 parts, among them J1 128x64 OLED Display, SW1 SW_Nidec_CAS-120A1, U1 AD8317_Module, U2 MT3608_Boost_converter, U3 ESP32-WEMOS D1 mini

Commit message: feat(Hw):Added_microcontroller
Parts:
- added C1: .1uF, Capacitor_SMD:C_0603_1608Metric, B.Cu at (155.0, 81.0)
- added C2: .1uF, Capacitor_SMD:C_0603_1608Metric, F.Cu at (82.4, 88.1)
- added D2: LED, LED_SMD:LED_0603_1608Metric, F.Cu at (86.4, 85.6)
- added D3: LED, LED_SMD:LED_0603_1608Metric, F.Cu at (86.4, 88.2)
- added D4: LED, LED_SMD:LED_0603_1608Metric, F.Cu at (86.4, 90.8)
- added D5: LED, LED_SMD:LED_0603_1608Metric, F.Cu at (86.4, 93.4)
- added D6: LED, LED_SMD:LED_0603_1608Metric, F.Cu at (86.4, 96.0)
- added D7: R_LED, badge-44con-2025:LYT77K-K2M1, F.Cu at (93.0, 102.0)
- added D8: R_LED, badge-44con-2025:LYT77K-K2M1, F.Cu at (90.0, 106.0)
- added J2: Conn_02x03_Odd_Even, Connector_PinHeader_2.54mm:PinHeader_2x03_P2.54mm_Vertical_SMD, F.Cu at (112.0, 50.0)
- added R2: 220, Resistor_SMD:R_0603_1608Metric, F.Cu at (82.4, 90.6)
- added R3: 220, Resistor_SMD:R_0603_1608Metric, F.Cu at (82.4, 93.1)
- added R4: 220, Resistor_SMD:R_0603_1608Metric, F.Cu at (82.4, 95.6)
- added R5: 220, Resistor_SMD:R_0603_1608Metric, F.Cu at (82.4, 98.1)
- added R6: 220, Resistor_SMD:R_0603_1608Metric, F.Cu at (82.4, 100.6)
- added R7: 220, Resistor_SMD:R_0603_1608Metric, F.Cu at (82.4, 103.2)
- added R8: 220, Resistor_SMD:R_0603_1608Metric, F.Cu at (82.4, 105.7)
- added SW1: RESET, Button_Switch_SMD:SW_SPST_TL3342, F.Cu at (122.9, 78.1)
- added U2: CH32V003FxPx, Package_SO:TSSOP-20_4.4x6.5mm_P0.65mm, B.Cu at (157.0, 75.0)
- moved BT3 123.7 mm to (197.2, 140.4), turned to 90 degrees
- moved U4 120.4 mm to (204.4, 44.2), turned to -90 degrees
- moved SW2 91.7 mm to (202.1, 86.6), turned to -90 degrees
- moved U3 88.0 mm to (124.5, 109.8)
- moved U1 49.1 mm to (138.3, 96.4), turned to 90 degrees
- moved BT2 44.1 mm to (183.2, 95.7), turned to -90 degrees
- moved BT1 36.1 mm to (169.1, 95.7), turned to -90 degrees
- moved RV1 15.0 mm to (151.0, 125.0), turned to 180 degrees
- moved J1 13.2 mm to (157.1, 75.0)
- moved JP1 12.7 mm to (181.1, 84.5)
- moved BZ1 9.54 mm to (127.5, 121.0)
- moved D1 9.24 mm to (140.3, 136.0)
- moved R1 9.24 mm to (140.2, 138.6)
- renumbered BT7 to BT1, BT5 to BT2, BT6 to BT3, D7 to D1, R4 to R1, SW1 to SW2, U3 to U1, U2 to U3, U1 to U4
Other:
- board size 80.2 x 100 mm -> 100 x 100 mm

Commit message: fix(Hw): Changed_PCB_design
Parts:
- removed D6: LED, LED_SMD:LED_0603_1608Metric
- removed D7, D8: R_LED, badge-44con-2025:LYT77K-K2M1
- removed R6, R7, R8: 220, Resistor_SMD:R_0603_1608Metric
- RV1: footprint Potentiometer_THT:Potentiometer_Alps_RK163_Single_Horizontal -> badge-44con-2025:Potentiometer_generic; moved to B.Cu
- U4: moved to F.Cu
- moved SW2 97.5 mm to (109.7, 117.8)
- moved R3 77.2 mm to (156.1, 116.1), turned to 90 degrees
- moved D3 73.5 mm to (154.4, 116.1), turned to 90 degrees
- moved R2 71.3 mm to (143.1, 128.0)
- moved D2 69.8 mm to (143.1, 126.4)
- moved R4 61.6 mm to (143.3, 105.0)
- moved D4 59.0 mm to (143.3, 106.6)
- moved R5 54.2 mm to (132.4, 119.1), turned to -90 degrees
- moved D5 51.2 mm to (132.4, 115.9), turned to 90 degrees
- moved C2 43.2 mm to (125.5, 86.1)
- moved U4 37.1 mm to (167.8, 50.2)
- moved R1 33.8 mm to (109.8, 123.8)
- moved D1 32.3 mm to (109.8, 125.4), turned to 180 degrees
- moved U3 15.9 mm to (139.8, 105.6), turned to 180 degrees
- moved JP1 15.4 mm to (195.1, 78.2)
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Connections:
- J1 pad 1: /SDA -> /SDA_ESP
- J1 pad 2: /SCL -> /SCL_ESP
- R2 pad 2: GND -> Net-(R2-Pad2)
- R3 pad 2: GND -> Net-(R2-Pad2)
- R4 pad 2: GND -> Net-(R2-Pad2)
- R5 pad 2: GND -> Net-(R2-Pad2)
- U1 pad 23: /SCL -> /SCL_ESP
- U1 pad 24: /SDA -> /SDA_ESP
- U2 pad 13: /LEFT -> unconnected-(U2-PC3-Pad13)
- U2 pad 14: /UP -> unconnected-(U2-PC4-Pad14)
- U2 pad 6: /DOWN -> unconnected-(U2-PA2-Pad6)
- U2 pad 8: /RIGHT -> unconnected-(U2-PD0-Pad8)
Other:
- outline, holes or cut-outs redrawn

Commit message: feat(Hw): Started routing
Parts:
- moved BT1 44.6 mm to (170.0, 137.1), turned to 90 degrees
- moved C2 11.8 mm to (122.7, 97.6)
- moved SW1 11.2 mm to (125.5, 92.8)
- moved D1 7.14 mm to (116.7, 127.2)
- moved R1 7.14 mm to (116.7, 125.6)
- moved RV1 2.71 mm to (143.2, 114.1)
- moved U3 1.01 mm to (140.3, 106.5)
- turned SW2 to 90 degrees
Routing:
- net +5V: track 0.00 -> 85.5 mm
- net +5VP: track 0.00 -> 77.1 mm
- net Net-(BT1--): track 0.00 -> 14.2 mm
- net Net-(BT2--): track 0.00 -> 14.0 mm
Other:
- outline, holes or cut-outs redrawn

Commit message: feat(Hw): finished_routing
Parts:
- added JP2: Jumper_3_Open, Jumper:SolderJumper-3_P1.3mm_Open_RoundedPad1.0x1.5mm, B.Cu at (158.6, 54.4)
- added JP3: Jumper_3_Open, Jumper:SolderJumper-3_P1.3mm_Open_RoundedPad1.0x1.5mm, B.Cu at (153.0, 54.3)
- D1: moved to B.Cu
- moved D1 19.6 mm to (110.5, 108.6), turned to 0 degrees
- moved R1 18.1 mm to (110.5, 108.6), turned to 180 degrees
- moved U2 2.25 mm to (153.5, 71.6)
- moved C1 1.48 mm to (151.7, 76.3)
- moved C2 1.00 mm to (122.7, 96.6), turned to 180 degrees
Connections:
- J1 pad 1: /SDA_ESP -> /SDA
- J1 pad 2: /SCL_ESP -> /SCL
- R2 pad 2: Net-(R2-Pad2) -> GND
- R3 pad 2: Net-(R2-Pad2) -> GND
- R4 pad 2: Net-(R2-Pad2) -> GND
- R5 pad 2: Net-(R2-Pad2) -> GND
- U2 pad 1: /LED3 -> /LED2
- U2 pad 10: /LED7 -> unconnected-(U2-PC0-Pad10)
- U2 pad 11: /SDA -> /CH3_SDA
- U2 pad 12: /SCL -> /CH3_SCL
- U2 pad 15: /LED6 -> unconnected-(U2-PC5-Pad15)
- U2 pad 19: /LED5 -> unconnected-(U2-PD2-Pad19)
- U2 pad 2: /LED2 -> /LED1
- U2 pad 20: /LED1 -> unconnected-(U2-PD3-Pad20)
- U2 pad 3: unconnected-(U2-PD6-Pad3) -> /LED3
Routing:
- net +3.3V: track 0.00 -> 155.9 mm, vias 0 -> 3
- net +9V: track 0.00 -> 98.0 mm, vias 0 -> 9
- net /POT: track 0.00 -> 79.4 mm
- net /LED1: track 0.00 -> 61.4 mm, vias 0 -> 1
- net /SDA_ESP: track 0.00 -> 58.6 mm, vias 0 -> 1
- net /LED4: track 0.00 -> 58.0 mm, vias 0 -> 3
- net /BUZZER: track 0.00 -> 57.7 mm, vias 0 -> 2
- net /SWDIO: track 0.00 -> 52.9 mm, vias 0 -> 1
- net /RST: track 0.00 -> 52.6 mm, vias 0 -> 1
- net /SCL_ESP: track 0.00 -> 46.2 mm
- net /LED2: track 0.00 -> 41.6 mm, vias 0 -> 1
- net /LED3: track 0.00 -> 40.8 mm, vias 0 -> 1
- net /AD8317_OUT: track 0.00 -> 36.5 mm
- net /CH3_SDA: track 0.00 -> 22.2 mm
- net /CH3_SCL: track 0.00 -> 19.2 mm, vias 0 -> 2
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- added copper zone on B.Cu, net +9V
- added copper zone on F.Cu, net +9V
- added copper zone on B.Cu, net GND
- added copper zone on F.Cu, net GND

Commit message: fix(Hw):fixed_BOM
Parts:
- moved J2 0.17 mm to (122.8, 55.5), turned to -90 degrees
Routing:
- net +3.3V: track 155.9 -> 165.7 mm
- net /SWDIO: track 52.9 -> 50.6 mm
